Commit message: four_wheel RSP is not being published

File: description/gazebo_control.xacro (robot description, xacro)
@@ -2,4 +2,8 @@
 <robot xmlns:xacro="http://www.ros.org/wiki/xacro">
     <!-- Robot Variables -->
+    <xacro:property name="chassis_length" value="0.35" />
+    <xacro:property name="chassis_width" value="0.3" />
+    <xacro:property name="chassis_height" value="0.08" />
+    <xacro:property name="chassis_mass" value="4.0" />
     <xacro:property name="wheel_radius" value="0.05" />
     <xacro:property name="wheel_thickness" value="0.018" />

File: description/ros2_control.xacro (robot description, xacro)
@@ -91,5 +91,5 @@
     </xacro:if>
     <!-- Gazebo plugin for ROS2 control -->
-    <gazebo>
+    <!-- <gazebo>
         <plugin name="gz_ros2_control::GazeboSimROS2ControlPlugin"
             filename="libgz_ros2_control-system.so">
@@ -97,4 +97,9 @@
             <parameters>$(find khepa_bot)/config/gaz_ros2_ctl_use_sim.yaml</parameters>
         </plugin>
+    </gazebo> -->
+    <gazebo>
+        <plugin name="gz::sim::systems::Ros2Control"
+            filename="libgz_ros2_control-system.so">
+        </plugin>
     </gazebo>
 </robot>
